File: Hardware/delay.kicad_sch (KiCad schematic)
At the start: 76 parts, among them Q7 MMBF5457, Q8 MMBT5088LT1G, Q9 MMBT5088LT1G, SW2 SW_DPDT_x2, U13 TL074, U18 TL074, U19 PT2399

Commit message: Add tap tempo smoothing
Added smoothing to the (soon to be added) tap tempo for the delay fx
Parts:
- removed TIME: B50k, symbol Device:R_Potentiometer
- added C157, C158: 1u, symbol Device:C
- added Q10: MMBT5088LT1G, Package_TO_SOT_SMD:SOT-23, symbol custom_parts:MMBT5088LT1G
- added R192: 18k, symbol Device:R
- added R193, R194: 100k, symbol Device:R
- added unit 3 of U18
- C143: value 100n -> 220n
- PRE1: value B100k -> B50k
- R174: value 4k7 -> 1k5
- R180: value 1k -> 5k6
- R181: value 1k -> 2k2
Connections:
- net GND: now also R174.2, C158.2, R193.2; no longer R174.1
- net MOD: no longer R174.2
- net at C133.1, R169.1, R170.2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: now also R192.2; no longer MIX.2
- net Pin6: now reaches U19.6 (VCO)
- net Pin6: now also Q10.3 (C)
- new net: C157.1, MIX.2
- new net: C157.2, R192.1
- new net: C158.1, R193.1, R194.2, U18.10 (+)
- new net: Q10.1 (B), U18.8
- new net: Q10.2 (E), R174.1, U18.9 (-)
- new net PWM In: R194.1
Other:
- moved on the sheet: C132, C133, C134, C135, C136, C137, C138, C139, C140, C141, C142, C143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
